File: usb_to_uart_converter.kicad_pcb (KiCad board)
At the start: 2 copper layers, 73 x 36.5 mm, 19 parts, among them J1 USB_B, J2 Jumper, J4 UART Output, U1 FT232RL

Commit message: update cleaner tracks
Parts:
- J1: footprint Connector_USB:USB_B_Amphenol_MUSB-D511_Vertical_Rugged -> my_USB_Connectors:USB_B_Amphenol_MUSB-D511_Vertical_Rugged
- moved C7 41.3 mm to (151.0, 113.5)
- moved J2 37.3 mm to (113.5, 126.0), turned to -90 degrees
- moved C2 35.2 mm to (123.2, 135.5), turned to 0 degrees
- moved J1 32.9 mm to (153.8, 132.3)
- moved R1 28.3 mm to (130.0, 135.0), turned to -90 degrees
- moved C6 26.4 mm to (137.5, 116.0), turned to 90 degrees
- moved FB1 26.2 mm to (147.0, 117.5), turned to 180 degrees
- moved C1 25.6 mm to (128.5, 122.0)
- moved C3 20.4 mm to (137.0, 121.0), turned to 180 degrees
- moved J4 20.0 mm to (128.5, 140.5)
- moved R3 18.3 mm to (128.2, 111.4), turned to 180 degrees
- moved R2 17.8 mm to (123.7, 111.4)
- moved U1 16.6 mm to (125.4, 128.1)
- moved D1 15.4 mm to (128.2, 115.4)
- moved D2 12.5 mm to (123.7, 115.4), turned to 90 degrees
Connections:
- net Net-(J1-D+) renamed /D+
- net Net-(J1-D-) renamed /D-
Routing:
- net /VCC: track 83.7 -> 48.7 mm, vias 2 -> 0
- net Net-(J1-VBUS): track 57.1 -> 22.9 mm
- net Net-(U1-CBUS3): track 22.9 -> 2.93 mm, vias 2 -> 0
- net GND: track 27.8 -> 20.2 mm, vias 9 -> 10
- net /D+: track 35.6 -> 30.0 mm, vias 2 -> 0
- net Net-(D2-K): track 13.1 -> 8.05 mm, vias 0 -> 2
- net VCCIO: track 66.8 -> 71.2 mm
- net /D-: track 34.2 -> 30.7 mm, vias 2 -> 0
- net Net-(D1-K): track 5.76 -> 9.28 mm, vias 0 -> 2
- net Net-(J4-Pin_4): track 11.8 -> 8.79 mm, vias 2 -> 0
- net Net-(J4-Pin_6): track 11.6 -> 14.2 mm, vias 0 -> 2
- net Net-(J4-Pin_2): track 11.2 -> 9.38 mm, vias 2 -> 0
- net Net-(D1-A): track 4.63 -> 2.81 mm
- net Net-(D2-A): track 4.41 -> 2.81 mm
- net Net-(J4-Pin_5): track 12.1 -> 13.2 mm, vias 1 -> 2
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Other:
- board text added: "V2.2"
- board text removed: "V2.1"
