File: usb_to_uart_converter.kicad_sch (KiCad schematic)
At the start: 19 parts, among them J1 USB_B, J2 Jumper, J4 UART Output, U1 FT232RL

Commit message: update cleaner tracks
Parts:
- J1: footprint Connector_USB:USB_B_Amphenol_MUSB-D511_Vertical_Rugged -> my_USB_Connectors:USB_B_Amphenol_MUSB-D511_Vertical_Rugged
Connections:
- net D-: now reaches J1.2 (D-), U1.16 (USBD-)
- net D+: now reaches J1.3 (D+), U1.15 (USBD+)
Other:
- note added: "match impedance for differential"
- moved on the sheet: C3, C6
Changed lines of the file:
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@@
 		(rev "2.1")
+	)
+	(text "match impedance\nfor differential"
+		(exclude_from_sim no)
+		(at 68.834 99.06 0)
+		(effects
+			(font
+				(size 1.27 1.27)
+			)
+		)
 	)
 	(text "Mounting holes without connection for housing"
@@
 	)
 	(junction
+		(at 96.52 55.88)
+		(diameter 0)
+		(color 0 0 0 0)
+	)
+	(junction
 		(at 109.22 119.38)
 		(diameter 0)
@@
 	)
 	(junction
-		(at 88.9 71.12)
-		(diameter 0)
-		(color 0 0 0 0)
-	)
-	(junction
 		(at 76.2 76.2)
 		(diameter 0)
@@
 	)
 	(junction
-		(at 85.09 110.49)
+		(at 92.71 35.56)
 		(diameter 0)
 		(color 0 0 0 0)
@@
 	)
 	(junction
-		(at 81.28 118.11)
+		(at 88.9 43.18)
 		(diameter 0)
 		(color 0 0 0 0)
@@
 	(wire
 		(pts
-			(xy 88.9 71.12) (xy 88.9 110.49)
-		)
-		(stroke
-			(width 0)
-			(type default)
-		)
-	)
-	(wire
-		(pts
 			(xy 190.5 104.14) (xy 194.31 104.14)
 		)
@@
 	(wire
 		(pts
-			(xy 76.2 118.11) (xy 81.28 118.11)
+			(xy 83.82 43.18) (xy 88.9 43.18)
 		)
 		(stroke
@@
 	(wire
 		(pts
-			(xy 85.09 115.57) (xy 85.09 118.11)
+			(xy 92.71 40.64) (xy 92.71 43.18)
 		)
 		(stroke
@@
 	(wire
 		(pts
-			(xy 76.2 110.49) (xy 85.09 110.49)
-		)
-		(stroke
-			(width 0)
-			(type default)
-		)
-	)
-	(wire
-		(pts
-			(xy 81.28 118.11) (xy 85.09 118.11)
+			(xy 83.82 35.56) (xy 92.71 35.56)
+		)
+		(stroke
+			(width 0)
+			(type default)
+		)
+	)
+	(wire
+		(pts
+			(xy 88.9 43.18) (xy 92.71 43.18)
 		)
 		(stroke
@@
 	(wire
 		(pts
-			(xy 88.9 55.88) (xy 135.89 55.88)
+			(xy 88.9 55.88) (xy 96.52 55.88)
 		)
 		(stroke
@@
 	(wire
 		(pts
+			(xy 96.52 55.88) (xy 135.89 55.88)
+		)
+		(stroke
+			(width 0)
+			(type default)
+		)
+	)
+	(wire
+		(pts
 			(xy 153.67 101.6) (xy 162.56 101.6)
 		)
@@
 	(wire
 		(pts
+			(xy 96.52 35.56) (xy 96.52 55.88)
+		)
+		(stroke
+			(width 0)
+			(type default)
+		)
+	)
+	(wire
+		(pts
 			(xy 153.67 81.28) (xy 158.75 81.28)
 		)
@@
 	(wire
 		(pts
-			(xy 76.2 115.57) (xy 76.2 118.11)
+			(xy 83.82 40.64) (xy 83.82 43.18)
 		)
 		(stroke
@@
 	(wire
 		(pts
-			(xy 85.09 110.49) (xy 88.9 110.49)
+			(xy 92.71 35.56) (xy 96.52 35.56)
 		)
 		(stroke
@@
 	(label "VCC"
 		(at 135.89 63.5 90)
+		(effects
+			(font
+				(size 1.27 1.27)
+			)
+			(justify left bottom)
+		)
+	)
+	(label "D-"
+		(at 54.61 104.14 0)
+		(effects
+			(font
+				(size 1.27 1.27)
+			)
+			(justify left bottom)
+		)
+	)
+	(label "D+"
+		(at 54.61 101.6 0)
 		(effects
 			(font
@@
 			)
 		)
-		(property "Footprint" "Connector_USB:USB_B_Amphenol_MUSB-D511_Vertical_Rugged"
+		(property "Footprint" "my_USB_Connectors:USB_B_Amphenol_MUSB-D511_Vertical_Rugged"
 			(at 48.26 102.87 0)
 			(effects
@@
 	(symbol
 		(lib_id "PCM_SparkFun-Capacitor:10uF_0603_6.3V_20%_Polar(Tant)")
-		(at 76.2 113.03 0)
+		(at 83.82 38.1 0)
 		(unit 1)
 		(exclude_from_sim no)
@@
 		(dnp no)
 		(property "Reference" "C6"
-			(at 70.104 109.728 0)
+			(at 77.724 34.798 0)
 			(effects
 				(font
@@
 		)
 		(property "Value" "10uF"
-			(at 70.104 112.268 0)
+			(at 77.724 37.338 0)
 			(effects
 				(font
@@
 		)
 		(property "Footprint" "PCM_SparkFun-Capacitor:C_0603_1608Metric_Polar"
-			(at 76.2 133.35 0)
+			(at 83.82 58.42 0)
 			(effects
 				(font
@@
 		)
 		(property "Datasheet" "https://datasheets.kyocera-avx.com/tc-series.pdf"
-			(at 77.47 128.27 0)
+			(at 85.09 53.34 0)
 			(effects
 				(font
@@
 		)
 		(property "Description" "Capacitor Tantalum 10uF 6.3V +/-20% 0603"
-			(at 76.2 130.81 0)
+			(at 83.82 55.88 0)
 			(effects
 				(font
@@
 		)
 		(property "PROD_ID" "CAP-13210"
-			(at 76.2 125.73 0)
+			(at 83.82 50.8 0)
 			(effects
 				(font
@@
 		)
 		(property "Voltage" "6.3V"
-			(at 70.104 114.808 0)
+			(at 77.724 39.878 0)
 			(effects
 				(font
@@
 		)
 		(property "Tolerance" "20%"
-			(at 70.104 117.348 0)
+			(at 77.724 42.418 0)
 			(effects
 				(font
@@
 	(symbol
 		(lib_id "PCM_SparkFun-Capacitor:0.1uF_0402_16V_10%")
-		(at 85.09 113.03 0)
+		(at 92.71 38.1 0)
 		(unit 1)
 		(exclude_from_sim no)
@@
 		(dnp no)
 		(property "Reference" "C3"
-			(at 89.408 109.728 0)
+			(at 97.028 34.798 0)
 			(effects
 				(font
@@
 		)
 		(property "Value" "0.1uF"
-			(at 87.63 111.7662 0)
+			(at 95.25 36.8362 0)
 			(effects
 				(font
@@
 		)
 		(property "Footprint" "PCM_SparkFun-Capacitor:C_0402_1005Metric"
-			(at 85.09 124.46 0)
+			(at 92.71 49.53 0)
 			(effects
 				(font
@@
 		)
 		(property "Datasheet" "https://cdn.sparkfun.com/assets/8/a/4/a/5/Kemet_Capacitor_Datasheet.pdf"
-			(at 85.09 127 0)
+			(at 92.71 52.07 0)
 			(effects
 				(font
@@
 		)
 		(property "Description" "Unpolarized capacitor"
-			(at 85.09 132.08 0)
+			(at 92.71 57.15 0)
 			(effects
 				(font
@@
 		)
 		(property "PROD_ID" "CAP-25565"
-			(at 85.09 129.54 0)
+			(at 92.71 54.61 0)
 			(effects
 				(font
@@
 		)
 		(property "Voltage" "16V"
-			(at 87.63 114.3062 0)
+			(at 95.25 39.3762 0)
 			(effects
 				(font
@@
 		)
 		(property "Tolerance" "10%"
-			(at 87.63 116.8462 0)
+			(at 95.25 41.9162 0)
 			(effects
 				(font
@@
 	(symbol
 		(lib_id "PCM_SparkFun-PowerSymbol:GND")
-		(at 81.28 118.11 0)
+		(at 88.9 43.18 0)
 		(unit 1)
 		(exclude_from_sim no)
@@
 		(fields_autoplaced yes)
 		(property "Reference" "#PWR04"
-			(at 81.28 124.46 0)
+			(at 88.9 49.53 0)
 			(effects
 				(font
@@
 		)
 		(property "Value" "GND"
-			(at 81.28 121.92 0)
+			(at 88.9 46.99 0)
 			(do_not_autoplace yes)
 			(effects
@@
 		)
 		(property "Footprint" ""
-			(at 81.28 118.11 0)
+			(at 88.9 43.18 0)
 			(effects
 				(font
@@
 		)
 		(property "Datasheet" ""
-			(at 81.28 118.11 0)
+			(at 88.9 43.18 0)
 			(effects
 				(font
@@
 		)
 		(property "Description" "Power symbol creates a global label with name \"GND\" , ground"
-			(at 81.28 127 0)
-			(effects
-				(font
+			(at 88.9 52.07 0)
+			(effects
+				(font
